Commit message: changes proposed to remove multiple terminal warnings

File: sr_description/arm/xacro/hand_support/shadowarm_handsupport_motor.transmission.xacro (robot description, xacro)
@@ -11,5 +11,5 @@
       </actuator>
       <joint name="ElbowJRotate">
-        <hardwareInterface>EffortJointInterface</hardwareInterface>
+        <hardwareInterface>hardware_interface/EffortJointInterface</hardwareInterface>
       </joint>
     </transmission>

File: sr_description/arm/xacro/hand_support/shadowarm_handsupport_muscle.transmission.xacro (robot description, xacro)
@@ -11,5 +11,5 @@
       </actuator>
       <joint name="ElbowJRotate">
-        <hardwareInterface>EffortJointInterface</hardwareInterface>
+        <hardwareInterface>hardware_interface/EffortJointInterface</hardwareInterface>
       </joint>
     </transmission>

File: sr_description/arm/xacro/lower_arm/shadowarm_lowerarm.transmission.xacro (robot description, xacro)
@@ -11,5 +11,5 @@
       </actuator>
       <joint name="ElbowJSwing">
-        <hardwareInterface>EffortJointInterface</hardwareInterface>
+        <hardwareInterface>hardware_interface/EffortJointInterface</hardwareInterface>
       </joint>
     </transmission>

File: sr_description/arm/xacro/trunk/shadowarm_trunk.transmission.xacro (robot description, xacro)
@@ -11,5 +11,5 @@
       </actuator>
       <joint name="ShoulderJRotate">
-        <hardwareInterface>EffortJointInterface</hardwareInterface>
+        <hardwareInterface>hardware_interface/EffortJointInterface</hardwareInterface>
       </joint>
     </transmission>

File: sr_description/arm/xacro/upper_arm/shadowarm_upperarm.transmission.xacro (robot description, xacro)
@@ -11,5 +11,5 @@
       </actuator>
       <joint name="ShoulderJSwing">
-        <hardwareInterface>EffortJointInterface</hardwareInterface>
+        <hardwareInterface>hardware_interface/EffortJointInterface</hardwareInterface>
       </joint>
     </transmission>

File: sr_description/hand/xacro/finger/distal/distal.transmission.xacro (robot description, xacro)
@@ -17,6 +17,6 @@
             </actuator>
             <joint name="${prefix}${joint_prefix}J1">
-                <hardwareInterface>EffortJointInterface</hardwareInterface>
-                <hardwareInterface>PositionJointInterface</hardwareInterface>
+                <hardwareInterface>hardware_interface/EffortJointInterface</hardwareInterface>
+                <hardwareInterface>hardware_interface/PositionJointInterface</hardwareInterface>
             </joint>
         </transmission>
@@ -30,6 +30,6 @@
             </actuator>
             <joint name="${prefix}${joint_prefix}J1">
-                <hardwareInterface>EffortJointInterface</hardwareInterface>
-                <hardwareInterface>PositionJointInterface</hardwareInterface>
+                <hardwareInterface>hardware_interface/EffortJointInterface</hardwareInterface>
+                <hardwareInterface>hardware_interface/PositionJointInterface</hardwareInterface>
             </joint>
         </transmission>

File: sr_description/hand/xacro/finger/knuckle/knuckle.transmission.xacro (robot description, xacro)
@@ -17,6 +17,6 @@
                 </actuator>
                 <joint name="${prefix}${joint_prefix}J4">
-                    <hardwareInterface>EffortJointInterface</hardwareInterface>
-                    <hardwareInterface>PositionJointInterface</hardwareInterface>
+                    <hardwareInterface>hardware_interface/EffortJointInterface</hardwareInterface>
+                    <hardwareInterface>hardware_interface/PositionJointInterface</hardwareInterface>
                 </joint>
             </transmission>
@@ -30,5 +30,5 @@
                 </actuator>
                 <joint name="${prefix}${joint_prefix}J4">
-                    <hardwareInterface>EffortJointInterface</hardwareInterface>
+                    <hardwareInterface>hardware_interface/EffortJointInterface</hardwareInterface>
                     <hardwareInterface>PositionJointInterface</hardwareInterface>
                 </joint>

File: sr_description/hand/xacro/finger/lfmetacarpal/lfmetacarpal.transmission.xacro (robot description, xacro)
@@ -15,6 +15,6 @@
                 </actuator>
                 <joint name="${prefix}LFJ5">
-                    <hardwareInterface>EffortJointInterface</hardwareInterface>
-                    <hardwareInterface>PositionJointInterface</hardwareInterface>
+                    <hardwareInterface>hardware_interface/EffortJointInterface</hardwareInterface>
+                    <hardwareInterface>hardware_interface/PositionJointInterface</hardwareInterface>
                 </joint>
             </transmission>
@@ -28,6 +28,6 @@
                 </actuator>
                 <joint name="${prefix}LFJ5">
-                    <hardwareInterface>EffortJointInterface</hardwareInterface>
-                    <hardwareInterface>PositionJointInterface</hardwareInterface>
+                    <hardwareInterface>hardware_interface/EffortJointInterface</hardwareInterface>
+                    <hardwareInterface>hardware_interface/PositionJointInterface</hardwareInterface>
                 </joint>
             </transmission>

File: sr_description/hand/xacro/finger/middle/middle.transmission.xacro (robot description, xacro)
@@ -17,10 +17,10 @@
                 </actuator>
                 <joint name="${prefix}${joint_prefix}J1">
-                    <hardwareInterface>EffortJointInterface</hardwareInterface>
-                    <hardwareInterface>PositionJointInterface</hardwareInterface>
+                    <hardwareInterface>hardware_interface/EffortJointInterface</hardwareInterface>
+                    <hardwareInterface>hardware_interface/PositionJointInterface</hardwareInterface>
                 </joint>
                 <joint name="${prefix}${joint_prefix}J2">
-                    <hardwareInterface>EffortJointInterface</hardwareInterface>
-                    <hardwareInterface>PositionJointInterface</hardwareInterface>
+                    <hardwareInterface>hardware_interface/EffortJointInterface</hardwareInterface>
+                    <hardwareInterface>hardware_interface/PositionJointInterface</hardwareInterface>
                 </joint>
                 <mechanicalReduction>1</mechanicalReduction>
@@ -35,6 +35,6 @@
                 </actuator>
                 <joint name="${prefix}${joint_prefix}J1">
-                    <hardwareInterface>EffortJointInterface</hardwareInterface>
-                    <hardwareInterface>PositionJointInterface</hardwareInterface>
+                    <hardwareInterface>hardware_interface/EffortJointInterface</hardwareInterface>
+                    <hardwareInterface>hardware_interface/PositionJointInterface</hardwareInterface>
                 </joint>
                 <secondJoint name="${prefix}${joint_prefix}J2"/>

File: sr_description/hand/xacro/finger/proximal/proximal.transmission.xacro (robot description, xacro)
@@ -17,6 +17,6 @@
                 </actuator>
                 <joint name="${prefix}${joint_prefix}J3">
-                    <hardwareInterface>EffortJointInterface</hardwareInterface>
-                    <hardwareInterface>PositionJointInterface</hardwareInterface>
+                    <hardwareInterface>hardware_interface/EffortJointInterface</hardwareInterface>
+                    <hardwareInterface>hardware_interface/PositionJointInterface</hardwareInterface>
                 </joint>
             </transmission>
@@ -30,6 +30,6 @@
                 </actuator>
                 <joint name="${prefix}${joint_prefix}J3">
-                    <hardwareInterface>EffortJointInterface</hardwareInterface>
-                    <hardwareInterface>PositionJointInterface</hardwareInterface>
+                    <hardwareInterface>hardware_interface/EffortJointInterface</hardwareInterface>
+                    <hardwareInterface>hardware_interface/PositionJointInterface</hardwareInterface>
                 </joint>
             </transmission>

File: sr_description/hand/xacro/forearm/forearm.urdf.xacro (robot description, xacro)
@@ -38,5 +38,5 @@
               <mesh filename="package://sr_description/meshes/hand/forearm.dae" scale="0.001 0.001 0.001" />
             </geometry>
-            <material name="light_grey" />
+            <xacro:light_grey/>
           </visual>
         </xacro:if>
@@ -47,5 +47,5 @@
               <mesh filename="package://sr_description/meshes/hand/forearm_visual_plus.dae" scale="0.001 0.001 0.001" />
             </geometry>
-            <material name="light_grey" />
+            <xacro:light_grey/>
           </visual>
         </xacro:if>

File: sr_description/hand/xacro/palm/palm.transmission.xacro (robot description, xacro)
@@ -15,6 +15,6 @@
                 </actuator>
                 <joint name="${prefix}WRJ1">
-                    <hardwareInterface>EffortJointInterface</hardwareInterface>
-                    <hardwareInterface>PositionJointInterface</hardwareInterface>
+                    <hardwareInterface>hardware_interface/EffortJointInterface</hardwareInterface>
+                    <hardwareInterface>hardware_interface/PositionJointInterface</hardwareInterface>
                 </joint>
             </transmission>
@@ -28,6 +28,6 @@
                 </actuator>
                 <joint name="${prefix}WRJ1">
-                    <hardwareInterface>EffortJointInterface</hardwareInterface>
-                    <hardwareInterface>PositionJointInterface</hardwareInterface>
+                    <hardwareInterface>hardware_interface/EffortJointInterface</hardwareInterface>
+                    <hardwareInterface>hardware_interface/PositionJointInterface</hardwareInterface>
                 </joint>
             </transmission>

File: sr_description/hand/xacro/thumb/thbase.transmission.xacro (robot description, xacro)
@@ -15,6 +15,6 @@
                 </actuator>
                 <joint name="${prefix}THJ5">
-                    <hardwareInterface>EffortJointInterface</hardwareInterface>
-                    <hardwareInterface>PositionJointInterface</hardwareInterface>
+                    <hardwareInterface>hardware_interface/EffortJointInterface</hardwareInterface>
+                    <hardwareInterface>hardware_interface/PositionJointInterface</hardwareInterface>
                 </joint>
             </transmission>
@@ -28,6 +28,6 @@
                 </actuator>
                 <joint name="${prefix}THJ5">
-                    <hardwareInterface>EffortJointInterface</hardwareInterface>
-                    <hardwareInterface>PositionJointInterface</hardwareInterface>
+                    <hardwareInterface>hardware_interface/EffortJointInterface</hardwareInterface>
+                    <hardwareInterface>hardware_interface/PositionJointInterface</hardwareInterface>
                 </joint>
             </transmission>

File: sr_description/hand/xacro/thumb/thdistal.transmission.xacro (robot description, xacro)
@@ -15,6 +15,6 @@
                 </actuator>
                 <joint name="${prefix}THJ1">
-                    <hardwareInterface>EffortJointInterface</hardwareInterface>
-                    <hardwareInterface>PositionJointInterface</hardwareInterface>
+                    <hardwareInterface>hardware_interface/EffortJointInterface</hardwareInterface>
+                    <hardwareInterface>hardware_interface/PositionJointInterface</hardwareInterface>
                 </joint>
             </transmission>
@@ -28,6 +28,6 @@
                 </actuator>
                 <joint name="${prefix}THJ1">
-                    <hardwareInterface>EffortJointInterface</hardwareInterface>
-                    <hardwareInterface>PositionJointInterface</hardwareInterface>
+                    <hardwareInterface>hardware_interface/EffortJointInterface</hardwareInterface>
+                    <hardwareInterface>hardware_interface/PositionJointInterface</hardwareInterface>
                 </joint>
             </transmission>

File: sr_description/hand/xacro/thumb/thhub.transmission.xacro (robot description, xacro)
@@ -15,6 +15,6 @@
                 </actuator>
                 <joint name="${prefix}THJ3">
-                    <hardwareInterface>EffortJointInterface</hardwareInterface>
-                    <hardwareInterface>PositionJointInterface</hardwareInterface>
+                    <hardwareInterface>hardware_interface/EffortJointInterface</hardwareInterface>
+                    <hardwareInterface>hardware_interface/PositionJointInterface</hardwareInterface>
                 </joint>
             </transmission>
@@ -28,5 +28,5 @@
                 </actuator>
                 <joint name="${prefix}THJ3">
-                    <hardwareInterface>EffortJointInterface</hardwareInterface>
+                    <hardwareInterface>hardware_interface/EffortJointInterface</hardwareInterface>
                     <hardwareInterface>PositionJointInterface</hardwareInterface>
                 </joint>

File: sr_description/hand/xacro/thumb/thmiddle.transmission.xacro (robot description, xacro)
@@ -15,6 +15,6 @@
                 </actuator>
                 <joint name="${prefix}THJ2">
-                    <hardwareInterface>EffortJointInterface</hardwareInterface>
-                    <hardwareInterface>PositionJointInterface</hardwareInterface>
+                    <hardwareInterface>hardware_interface/EffortJointInterface</hardwareInterface>
+                    <hardwareInterface>hardware_interface/PositionJointInterface</hardwareInterface>
                 </joint>
             </transmission>
@@ -28,6 +28,6 @@
                 </actuator>
                 <joint name="${prefix}THJ2">
-                    <hardwareInterface>EffortJointInterface</hardwareInterface>
-                    <hardwareInterface>PositionJointInterface</hardwareInterface>
+                    <hardwareInterface>hardware_interface/EffortJointInterface</hardwareInterface>
+                    <hardwareInterface>hardware_interface/PositionJointInterface</hardwareInterface>
                 </joint>
             </transmission>

File: sr_description/hand/xacro/thumb/thproximal.transmission.xacro (robot description, xacro)
@@ -15,6 +15,6 @@
                 </actuator>
                 <joint name="${prefix}THJ4">
-                    <hardwareInterface>EffortJointInterface</hardwareInterface>
-                    <hardwareInterface>PositionJointInterface</hardwareInterface>
+                    <hardwareInterface>hardware_interface/EffortJointInterface</hardwareInterface>
+                    <!--<hardwareInterface>hardware_interface/PositionJointInterface</hardwareInterface>-->
                 </joint>
             </transmission>
@@ -28,6 +28,6 @@
                 </actuator>
                 <joint name="${prefix}THJ4">
-                    <hardwareInterface>EffortJointInterface</hardwareInterface>
-                    <hardwareInterface>PositionJointInterface</hardwareInterface>
+                    <hardwareInterface>hardware_interface/EffortJointInterface</hardwareInterface>
+                    <!--<hardwareInterface>hardware_interface/PositionJointInterface</hardwareInterface>-->
                 </joint>
             </transmission>

File: sr_description/hand/xacro/wrist/wrist.transmission.xacro (robot description, xacro)
@@ -15,6 +15,6 @@
                 </actuator>
                 <joint name="${prefix}WRJ2">
-                    <hardwareInterface>EffortJointInterface</hardwareInterface>
-                    <hardwareInterface>PositionJointInterface</hardwareInterface>
+                    <hardwareInterface>hardware_interface/EffortJointInterface</hardwareInterface>
+                    <hardwareInterface>hardware_interface/PositionJointInterface</hardwareInterface>
                 </joint>
             </transmission>
@@ -28,6 +28,6 @@
                 </actuator>
                 <joint name="${prefix}WRJ2">
-                    <hardwareInterface>EffortJointInterface</hardwareInterface>
-                    <hardwareInterface>PositionJointInterface</hardwareInterface>
+                    <hardwareInterface>hardware_interface/EffortJointInterface</hardwareInterface>
+                    <hardwareInterface>hardware_interface/PositionJointInterface</hardwareInterface>
                 </joint>
             </transmission>
