Commit message: Add default values for virtual links
If no values are set for virtual links, PyBullet sets these values to 1, which
is undesired since it alters the robot's dynamics.

File: sr_description/hand/xacro/palm/imu.urdf.xacro (robot description, xacro)
@@ -1,5 +1,11 @@
 <robot xmlns:xacro="http://www.ros.org/wiki/xacro" name="shadowhand_motor">
   <xacro:macro name="imu_sensor" params="prefix">
-    <link name="${prefix}imu"/>
+    <link name="${prefix}imu">
+      <inertial>
+        <mass value="0.0"/>
+        <origin rpy="0 0 0" xyz="0 0 0"/>
+        <inertia ixx="0.0" ixy="0.0" ixz="0.0" iyy="0.0" iyz="0.0" izz="0.0"/>
+      </inertial>
+    </link>
     <joint name="${prefix}palm_to_imu" type="fixed">
       <parent link="${prefix}palm" />

File: sr_description/hand/xacro/palm/palm.urdf.xacro (robot description, xacro)
@@ -93,5 +93,11 @@
       <origin xyz="0.0 0.0 0.05" rpy="0.0 0.0 0.0" />
     </joint>
-    <link name="${prefix}manipulator" />
+    <link name="${prefix}manipulator">
+      <inertial>
+        <mass value="0.0"/>
+        <origin rpy="0 0 0" xyz="0 0 0"/>
+        <inertia ixx="0.0" ixy="0.0" ixz="0.0" iyy="0.0" iyz="0.0" izz="0.0"/>
+      </inertial>
+    </link>
     <joint name="${prefix}WRJ1" type="revolute">
       <parent link="${parent}" />

File: sr_description/hand/xacro/palm/palm_lite.urdf.xacro (robot description, xacro)
@@ -85,5 +85,11 @@
       <origin xyz="0.0 0.0 0.05" rpy="0.0 0.0 0.0" />
     </joint>
-    <link name="${prefix}manipulator" />
+    <link name="${prefix}manipulator">
+      <inertial>
+        <mass value="0.0"/>
+        <origin rpy="0 0 0" xyz="0 0 0"/>
+        <inertia ixx="0.0" ixy="0.0" ixz="0.0" iyy="0.0" iyz="0.0" izz="0.0"/>
+      </inertial>
+    </link>
     <!-- No wrist joints in a Lite palm -->
     <!-- extensions -->
